File: Ganglion_KiCad_Files/Ganglion_01.kicad_sch (KiCad schematic)
At the start: 92 parts, among them P1 CONN_02X08, P2 CONN_01X04, P3 CONN_01X04, P4 CONN_01X08, P5 CONN_01X08, SW1 CJS1200, SW2 CJS1200, SW3 CJS1200, SW4 CJS1200, SW5 SPDT, SW6 TACT_SWITCH, U10 NCP300, U11 NCP551, U2 AD8237, U25 MCP6V31U, U3 AD8237, U4 AD8237, U5 AD8237, U6 LM7332, U7 MCP3912, U8 rfd_77101, U9 NCP551, Y1 Crystal_Small

Commit message: Changed resistor footprints
Parts:
- R47, R49: footprint Resistors_SMD:R_0603 -> Resistor_SMD:R_0805_2012Metric_Pad1.20x1.40mm_HandSolder
Changed lines of the file:
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@@
     (effects (font (size 1.524 1.524)) (justify left bottom))
   )
-  (label "D_3|A_4" (at 381 132.08 0)
+  (label "D_3|A_4" (at 381 132.08 0) (fields_autoplaced)
     (effects (font (size 1.524 1.524)) (justify left bottom))
   )
-  (label "D_11" (at 198.12 196.85 0)
+  (label "D_11" (at 198.12 196.85 0) (fields_autoplaced)
     (effects (font (size 1.524 1.524)) (justify left bottom))
   )
-  (label "FACTORY" (at 198.12 176.53 0)
+  (label "FACTORY" (at 198.12 176.53 0) (fields_autoplaced)
     (effects (font (size 1.524 1.524)) (justify left bottom))
   )
-  (label "REF+_OUT" (at 158.75 99.06 0)
+  (label "REF+_OUT" (at 158.75 99.06 0) (fields_autoplaced)
     (effects (font (size 1.524 1.524)) (justify left bottom))
   )
-  (label "D_12" (at 379.73 170.18 0)
+  (label "D_12" (at 379.73 170.18 0) (fields_autoplaced)
     (effects (font (size 1.524 1.524)) (justify left bottom))
   )
-  (label "3_-IN" (at 57.15 149.86 0)
+  (label "3_-IN" (at 57.15 149.86 0) (fields_autoplaced)
     (effects (font (size 1.524 1.524)) (justify left bottom))
   )
-  (label "D_24" (at 302.26 189.23 180)
+  (label "D_24" (at 302.26 189.23 180) (fields_autoplaced)
     (effects (font (size 1.524 1.524)) (justify right bottom))
   )
-  (label "SIM_TX" (at 255.27 248.92 90)
+  (label "SIM_TX" (at 255.27 248.92 90) (fields_autoplaced)
     (effects (font (size 1.524 1.524)) (justify left bottom))
   )
-  (label "SIM_RX" (at 250.19 248.92 90)
+  (label "SIM_RX" (at 250.19 248.92 90) (fields_autoplaced)
     (effects (font (size 1.524 1.524)) (justify left bottom))
   )
-  (label "MOSI" (at 379.73 167.64 0)
+  (label "MOSI" (at 379.73 167.64 0) (fields_autoplaced)
     (effects (font (size 1.524 1.524)) (justify left bottom))
   )
-  (label "D_3|A_4" (at 247.65 248.92 90)
+  (label "D_3|A_4" (at 247.65 248.92 90) (fields_autoplaced)
     (effects (font (size 1.524 1.524)) (justify left bottom))
   )
-  (label "SIM_RST" (at 379.73 181.61 0)
+  (label "SIM_RST" (at 379.73 181.61 0) (fields_autoplaced)
     (effects (font (size 1.524 1.524)) (justify left bottom))
   )
-  (label "CLK" (at 379.73 165.1 0)
+  (label "CLK" (at 379.73 165.1 0) (fields_autoplaced)
     (effects (font (size 1.524 1.524)) (justify left bottom))
   )
-  (label "D_12" (at 198.12 194.31 0)
+  (label "D_12" (at 198.12 194.31 0) (fields_autoplaced)
     (effects (font (size 1.524 1.524)) (justify left bottom))
   )
-  (label "D_5|A_6" (at 381 134.62 0)
+  (label "D_5|A_6" (at 381 134.62 0) (fields_autoplaced)
     (effects (font (size 1.524 1.524)) (justify left bottom))
   )
-  (label "MCP_RST" (at 209.55 45.72 180)
+  (label "MCP_RST" (at 209.55 45.72 180) (fields_autoplaced)
     (effects (font (size 1.524 1.524)) (justify right bottom))
   )
-  (label "SIM_RX" (at 381 129.54 0)
+  (label "SIM_RX" (at 381 129.54 0) (fields_autoplaced)
     (effects (font (size 1.524 1.524)) (justify left bottom))
   )
-  (label "MCP_RST" (at 306.07 194.31 180)
+  (label "MCP_RST" (at 306.07 194.31 180) (fields_autoplaced)
     (effects (font (size 1.524 1.524)) (justify right bottom))
   )
-  (label "D_21" (at 379.73 198.12 0)
+  (label "D_21" (at 379.73 198.12 0) (fields_autoplaced)
     (effects (font (size 1.524 1.524)) (justify left bottom))
   )
-  (label "D_9" (at 198.12 199.39 0)
+  (label "D_9" (at 198.12 199.39 0) (fields_autoplaced)
     (effects (font (size 1.524 1.524)) (justify left bottom))
   )
-  (label "MCP_SS" (at 209.55 55.88 180)
+  (label "MCP_SS" (at 209.55 55.88 180) (fields_autoplaced)
     (effects (font (size 1.524 1.524)) (justify right bottom))
   )
-  (label "I_BIAS" (at 35.56 55.88 0)
+  (label "I_BIAS" (at 35.56 55.88 0) (fields_autoplaced)
     (effects (font (size 1.524 1.524)) (justify left bottom))
   )
-  (label "SIM_RST" (at 198.12 173.99 0)
+  (label "SIM_RST" (at 198.12 173.99 0) (fields_autoplaced)
     (effects (font (size 1.524 1.524)) (justify left bottom))
   )
-  (label "D_4|A_5" (at 379.73 184.15 0)
+  (label "D_4|A_5" (at 379.73 184.15 0) (fields_autoplaced)
     (effects (font (size 1.524 1.524)) (justify left bottom))
   )
-  (label "V_BATT" (at 285.75 64.77 0)
+  (label "V_BATT" (at 285.75 64.77 0) (fields_autoplaced)
     (effects (font (size 1.524 1.524)) (justify left bottom))
   )
-  (label "D_21" (at 302.26 186.69 180)
+  (label "D_21" (at 302.26 186.69 180) (fields_autoplaced)
     (effects (font (size 1.524 1.524)) (justify right bottom))
   )
-  (label "V_ENABLE" (at 271.78 39.37 0)
+  (label "V_ENABLE" (at 271.78 39.37 0) (fields_autoplaced)
     (effects (font (size 1.524 1.524)) (justify left bottom))
   )
-  (label "I_BIAS" (at 35.56 179.07 0)
+  (label "I_BIAS" (at 35.56 179.07 0) (fields_autoplaced)
     (effects (font (size 1.524 1.524)) (justify left bottom))
   )
-  (label "I_BIAS" (at 35.56 97.79 0)
+  (label "I_BIAS" (at 35.56 97.79 0) (fields_autoplaced)
     (effects (font (size 1.524 1.524)) (justify left bottom))
   )
-  (label "D_11" (at 381 139.7 0)
+  (label "D_11" (at 381 139.7 0) (fields_autoplaced)
     (effects (font (size 1.524 1.524)) (justify left bottom))
   )
-  (label "D_14" (at 379.73 179.07 0)
+  (label "D_14" (at 379.73 179.07 0) (fields_autoplaced)
     (effects (font (size 1.524 1.524)) (justify left bottom))
   )
-  (label "V_ENABLE" (at 347.98 39.37 0)
+  (label "V_ENABLE" (at 347.98 39.37 0) (fields_autoplaced)
     (effects (font (size 1.524 1.524)) (justify left bottom))
   )
-  (label "MCP_SS" (at 257.81 248.92 90)
+  (label "MCP_SS" (at 257.81 248.92 90) (fields_autoplaced)
     (effects (font (size 1.524 1.524)) (justify left bottom))
   )
-  (label "V_IN" (at 306.07 73.66 0)
+  (label "V_IN" (at 306.07 73.66 0) (fields_autoplaced)
     (effects (font (size 1.524 1.524)) (justify left bottom))
   )
-  (label "D_24" (at 379.73 195.58 0)
+  (label "D_24" (at 379.73 195.58 0) (fields_autoplaced)
     (effects (font (size 1.524 1.524)) (justify left bottom))
   )
-  (label "4_-IN" (at 57.15 190.5 0)
+  (label "4_-IN" (at 57.15 190.5 0) (fields_autoplaced)
     (effects (font (size 1.524 1.524)) (justify left bottom))
   )
-  (label "V_ENABLE" (at 318.77 71.12 0)
+  (label "V_ENABLE" (at 318.77 71.12 0) (fields_autoplaced)
     (effects (font (size 1.524 1.524)) (justify left bottom))
   )
-  (label "D_4|A_5" (at 306.07 196.85 180)
+  (label "D_4|A_5" (at 306.07 196.85 180) (fields_autoplaced)
     (effects (font (size 1.524 1.524)) (justify right bottom))
   )
-  (label "SCK" (at 379.73 160.02 0)
+  (label "SCK" (at 379.73 160.02 0) (fields_autoplaced)
     (effects (font (size 1.524 1.524)) (justify left bottom))
   )
-  (label "2_-IN" (at 57.15 109.22 0)
+  (label "2_-IN" (at 57.15 109.22 0) (fields_autoplaced)
     (effects (font (size 1.524 1.524)) (justify left bottom))
   )
-  (label "I_BIAS" (at 35.56 138.43 0)
+  (label "I_BIAS" (at 35.56 138.43 0) (fields_autoplaced)
     (effects (font (size 1.524 1.524)) (justify left bottom))
   )
-  (label "D_23" (at 379.73 186.69 0)
+  (label "D_23" (at 379.73 186.69 0) (fields_autoplaced)
     (effects (font (size 1.524 1.524)) (justify left bottom))
   )
-  (label "V_IN" (at 269.24 34.29 0)
+  (label "V_IN" (at 269.24 34.29 0) (fields_autoplaced)
     (effects (font (size 1.524 1.524)) (justify left bottom))
   )
-  (label "D_2|A_3" (at 252.73 248.92 90)
+  (label "D_2|A_3" (at 252.73 248.92 90) (fields_autoplaced)
     (effects (font (size 1.524 1.524)) (justify left bottom))
   )
-  (label "1_-IN" (at 57.15 67.31 0)
+  (label "1_-IN" (at 57.15 67.31 0) (fields_autoplaced)
     (effects (font (size 1.524 1.524)) (justify left bottom))
   )
-  (label "MISO" (at 379.73 157.48 0)
+  (label "MISO" (at 379.73 157.48 0) (fields_autoplaced)
     (effects (font (size 1.524 1.524)) (justify left bottom))
   )
-  (label "V_IN" (at 345.44 34.29 0)
+  (label "V_IN" (at 345.44 34.29 0) (fields_autoplaced)
     (effects (font (size 1.524 1.524)) (justify left bottom))
   )
-  (label "RST" (at 379.73 162.56 0)
+  (label "RST" (at 379.73 162.56 0) (fields_autoplaced)
     (effects (font (size 1.524 1.524)) (justify left bottom))
   )
-  (label "D_14" (at 265.43 248.92 90)
+  (label "D_14" (at 265.43 248.92 90) (fields_autoplaced)
     (effects (font (size 1.524 1.524)) (justify left bottom))
   )
-  (label "D_2|A_3" (at 381 127 0)
+  (label "D_2|A_3" (at 381 127 0) (fields_autoplaced)
     (effects (font (size 1.524 1.524)) (justify left bottom))
   )
-  (label "D_5|A_6" (at 245.11 248.92 90)
+  (label "D_5|A_6" (at 245.11 248.92 90) (fields_autoplaced)
     (effects (font (size 1.524 1.524)) (justify left bottom))
   )
-  (label "SIM_TX" (at 381 124.46 0)
+  (label "SIM_TX" (at 381 124.46 0) (fields_autoplaced)
     (effects (font (size 1.524 1.524)) (justify left bottom))
   )
-  (label "D_23" (at 302.26 191.77 180)
+  (label "D_23" (at 302.26 191.77 180) (fields_autoplaced)
     (effects (font (size 1.524 1.524)) (justify right bottom))
   )
-  (label "D_9" (at 381 137.16 0)
+  (label "D_9" (at 381 137.16 0) (fields_autoplaced)
     (effects (font (size 1.524 1.524)) (justify left bottom))
   )
@@
       (effects (font (size 1.27 1.27)))
     )
-    (property "Footprint" "Resistors_SMD:R_0603" (at 372.618 168.91 90)
+    (property "Footprint" "Resistor_SMD:R_0805_2012Metric_Pad1.20x1.40mm_HandSolder" (at 372.618 168.91 90)
       (effects (font (size 1.27 1.27)) hide)
     )
@@
       (effects (font (size 1.27 1.27)))
     )
-    (property "Footprint" "Resistors_SMD:R_0603" (at 120.65 221.742 90)
+    (property "Footprint" "Resistor_SMD:R_0805_2012Metric_Pad1.20x1.40mm_HandSolder" (at 120.65 221.742 90)
       (effects (font (size 1.27 1.27)) hide)
     )
