File: Ganglion_KiCad_Files/Ganglion_Sensors_01.kicad_sch (KiCad schematic)
At the start: 25 parts, among them U12 AD5621, U13 SEEED_microSD, U14 MCP6V13T, U15 MCP6001, U16 SN74LVC1G32, U17 LIS2DE12, U18 74LVC1G66, U19 74LVC1G66, U20 74LVC1G66, U21 74LVC1G66, U22 74LVC1G66, U23 74LVC2G00

Commit message: Changed resistor footprints
Parts:
- R41, R42, R43, R44, R45, R46: footprint Resistors_SMD:R_0603 -> Resistor_SMD:R_0805_2012Metric_Pad1.20x1.40mm_HandSolder
Changed lines of the file:
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@@
     (effects (font (size 1.524 1.524)) (justify left bottom))
   )
-  (label "IMP_SIG" (at 229.87 116.84 0)
+  (label "IMP_SIG" (at 229.87 116.84 0) (fields_autoplaced)
     (effects (font (size 1.524 1.524)) (justify left bottom))
   )
-  (label "IMP_SIG" (at 228.6 147.32 0)
+  (label "IMP_SIG" (at 228.6 147.32 0) (fields_autoplaced)
     (effects (font (size 1.524 1.524)) (justify left bottom))
   )
-  (label "IMP_SIG" (at 68.58 118.11 180)
+  (label "IMP_SIG" (at 68.58 118.11 180) (fields_autoplaced)
     (effects (font (size 1.524 1.524)) (justify right bottom))
   )
-  (label "IMP_SIG" (at 177.8 116.84 0)
+  (label "IMP_SIG" (at 177.8 116.84 0) (fields_autoplaced)
     (effects (font (size 1.524 1.524)) (justify left bottom))
   )
-  (label "IMP_SIG" (at 177.8 147.32 0)
+  (label "IMP_SIG" (at 177.8 147.32 0) (fields_autoplaced)
     (effects (font (size 1.524 1.524)) (justify left bottom))
   )
-  (label "IMP_SIG" (at 203.2 88.9 0)
+  (label "IMP_SIG" (at 203.2 88.9 0) (fields_autoplaced)
     (effects (font (size 1.524 1.524)) (justify left bottom))
   )
@@
       (effects (font (size 1.27 1.27)))
     )
-    (property "Footprint" "Resistors_SMD:R_0603" (at 74.93 107.442 90)
+    (property "Footprint" "Resistor_SMD:R_0805_2012Metric_Pad1.20x1.40mm_HandSolder" (at 74.93 107.442 90)
       (effects (font (size 1.27 1.27)) hide)
     )
@@
       (effects (font (size 1.27 1.27)))
     )
-    (property "Footprint" "Resistors_SMD:R_0603" (at 96.52 88.392 90)
+    (property "Footprint" "Resistor_SMD:R_0805_2012Metric_Pad1.20x1.40mm_HandSolder" (at 96.52 88.392 90)
       (effects (font (size 1.27 1.27)) hide)
     )
@@
       (effects (font (size 1.27 1.27)))
     )
-    (property "Footprint" "Resistors_SMD:R_0603" (at 96.52 107.442 90)
+    (property "Footprint" "Resistor_SMD:R_0805_2012Metric_Pad1.20x1.40mm_HandSolder" (at 96.52 107.442 90)
       (effects (font (size 1.27 1.27)) hide)
     )
@@
       (effects (font (size 1.27 1.27)))
     )
-    (property "Footprint" "Resistors_SMD:R_0603" (at 137.16 83.058 90)
+    (property "Footprint" "Resistor_SMD:R_0805_2012Metric_Pad1.20x1.40mm_HandSolder" (at 137.16 83.058 90)
       (effects (font (size 1.27 1.27)) hide)
     )
@@
       (effects (font (size 1.27 1.27)))
     )
-    (property "Footprint" "Resistors_SMD:R_0603" (at 141.732 95.25 90)
+    (property "Footprint" "Resistor_SMD:R_0805_2012Metric_Pad1.20x1.40mm_HandSolder" (at 141.732 95.25 90)
       (effects (font (size 1.27 1.27)) hide)
     )
@@
       (effects (font (size 1.27 1.27)))
     )
-    (property "Footprint" "Resistors_SMD:R_0603" (at 176.022 46.99 90)
-      (effects (font (size 1.27 1.27)) hide)
-    )
+    (property "Footprint" "Resistor_SMD:R_0805_2012Metric_Pad1.20x1.40mm_HandSolder" (at 176.022 46.99 90)
+      (effects (font (size 1.27 1.27)) hide)
+    )
