File: Ganglion_KiCad_Files/References.kicad_sch (KiCad schematic)
At the start: 20 parts, among them U1 MCP6V31U, U24 MCP6V31U, U26 MCP6V31U, U27 MCP6V31U

Commit message: Changed resistor footprints
Parts:
- R48: footprint Capacitors_SMD:C_0603 -> Resistor_SMD:R_0805_2012Metric_Pad1.20x1.40mm_HandSolder
Changed lines of the file:
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@@
       (effects (font (size 1.27 1.27)))
     )
-    (property "Footprint" "Capacitors_SMD:C_0603" (at 195.58 111.252 90)
+    (property "Footprint" "Resistor_SMD:R_0805_2012Metric_Pad1.20x1.40mm_HandSolder" (at 195.58 111.252 90)
       (effects (font (size 1.27 1.27)) hide)
     )
